File: hardware_kicad/shared-memory.kicad_sch (KiCad schematic)
At the start: 13 parts, among them U2 CH32V003FxPx, U3 CH32V003FxPx, U4 23LCV1024, U5 74LVC125, U6 74LVC125

Commit message: refactor(schematic): optimize bus handshake and add cross-reset capabilities
- Rename handshake control lines to ~{BUSREQ} and ~{BUS_GRANT}
- Update active-low reset labels to ~{M1_NRST} and ~{M2_NRST}
- Formally establish physical cross-reset connections between cores
- Add 4k7 pull-up resistors on shared bus control lines
- Move M2 BUS_EN control line to M1 for better hardware arbitration
Parts:
- added R10, R9: 4k7, symbol Device:R
Connections:
- net M1_NRST is gone; now on net ~{M1_NRST}: U2.4 (PD7)
- net M2_NRST is gone; now on net ~{M2_NRST}: U3.4 (PD7)
- net +3V3: now also R10.1, R9.1
- net ~{BUSREQ}: now also R9.2
- net ~{M1_BUS_EN}: now also U2.19 (PD2); no longer U2.13 (PC3)
- net ~{M2_BUS_EN}: now also U2.20 (PD3); no longer U3.13 (PC3)
- net ~{M2_NRST}: now reaches U2.1 (PD4)
- net ~{M1_NRST}: now reaches U3.1 (PD4)
- net ~{BUSACK} renamed ~{BUS_GRANT}
- net ~{BUS_GRANT}: now also R10.2
Other:
- moved on the sheet: R2, R6, R7, R8, U3, U6A, U6B, U6C, U6D, U6E
